File: esp8266-breakout-for-autoprogramming.kicad_pcb (KiCad board)
At the start: 2 copper layers, 33.7 x 36.4 mm, 16 parts, among them J1 Conn_01x06_Female, U1 ESP-12E_SMD

Commit message: cleanup
Parts:
- renumbered ADC to TP1, GPIO16 to TP2, GPIO14 to TP3, GPIO12 to TP4, GPIO13 to TP5, GPIO5 to TP6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

Commit message: Fixed ERC
Parts:
- U1: value ESP-12E_SMD -> ESP-12E
