File: esp8266-breakout-for-autoprogramming.sch (KiCad schematic (older format))
At the start: 16 parts, among them J1 Conn_01x06_Female, U1 ESP-12E

Commit message: Fixed ERC
Changed lines of the file:
@@
 	700  2200 700  2000
 Wire Wire Line
-	700  2000 900  2000
+	700  2000 850  2000
 Wire Wire Line
 	700  1150 700  1200
@@
 	6150 1400 6450 1400
 $Comp
-L power:+3V3 #PWR?
+L power:+3V3 #PWR0106
 U 1 1 5E0FBB7E
 P 6950 1600
-F 0 "#PWR?" H 6950 1450 50  0001 C CNN
+F 0 "#PWR0106" H 6950 1450 50  0001 C CNN
 F 1 "+3V3" H 6965 1773 50  0000 C CNN
 F 2 "" H 6950 1600 50  0001 C CNN
@@
 	1    0    0    -1
 $EndComp
+$Comp
+L power:PWR_FLAG #FLG0102
+U 1 1 5E103890
+P 850 2200
+F 0 "#FLG0102" H 850 2275 50  0001 C CNN
+F 1 "PWR_FLAG" H 850 2373 50  0000 C CNN
+F 2 "" H 850 2200 50  0001 C CNN
+F 3 "~" H 850 2200 50  0001 C CNN
+	1    850  2200
+	-1   0    0    1
+$EndComp
+Wire Wire Line
+	850  2000 850  2200
+Connection ~ 850  2000
+Wire Wire Line
+	850  2000 900  2000
 $EndSCHEMATC
